File: schematics/mic_extension_board/mic_extension_board.kicad_pcb (KiCad board)
At the start: 2 copper layers, 87 x 62.2 mm, 87 parts, among them J1 XLR3, J2 Conn_01x02_Male, J3 Aux In, J4 I2C Bus, J5 6Pin ISP, J6 Input/Output, J7 XLR3, J8 XLR3, J9 Conn_01x03_Female, SW1 Stompbutton 1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

Commit message: more layouting
Parts:
- removed J6: Input/Output, Connector_PinHeader_2.54mm:PinHeader_1x04_P2.54mm_Vertical
- added C10: 4.7uF, Capacitor_SMD:CP_Elec_4x4.5, F.Cu at (139.7, 93.3)
- added C18: 220pF, Capacitor_SMD:C_0603_1608Metric_Pad1.08x0.95mm_HandSolder, F.Cu at (139.7, 85.5)
- added C19: 1uF, Capacitor_SMD:CP_Elec_4x4.5, F.Cu at (136.0, 80.6)
- added C20: 1uF, Capacitor_SMD:CP_Elec_4x4.5, F.Cu at (121.2, 97.8)
- added C21: 4.7uF, Capacitor_SMD:CP_Elec_4x4.5, F.Cu at (83.8, 36.8)
- added C22: 4.7uF, Capacitor_SMD:CP_Elec_4x4.5, F.Cu at (90.8, 36.7)
- added C23: 10uF, Capacitor_SMD:CP_Elec_4x4.5, F.Cu at (185.8, 82.5)
- added C24: 0.1uF, Capacitor_SMD:C_1210_3225Metric_Pad1.33x2.70mm_HandSolder, F.Cu at (161.3, 83.8)
- added C25: 10uF, Capacitor_SMD:CP_Elec_4x4.5, F.Cu at (191.1, 94.0)
- added C26: 0.1uF, Capacitor_SMD:C_1210_3225Metric_Pad1.33x2.70mm_HandSolder, F.Cu at (161.9, 78.7)
- added C27: 220pF, Capacitor_SMD:C_0603_1608Metric_Pad1.08x0.95mm_HandSolder, F.Cu at (177.8, 85.7)
- added C28: 220pF, Capacitor_SMD:C_0603_1608Metric_Pad1.08x0.95mm_HandSolder, F.Cu at (184.7, 77.5)
- added C29: 3.3uF, Capacitor_SMD:CP_Elec_4x4.5, F.Cu at (172.4, 75.6)
- added C30: 3.3uF, Capacitor_SMD:CP_Elec_4x4.5, F.Cu at (178.1, 94.6)
- added C31: 0.1uF, Capacitor_SMD:C_1210_3225Metric_Pad1.33x2.70mm_HandSolder, F.Cu at (178.4, 78.7)
- added C32: 47uF, Capacitor_SMD:CP_Elec_5x5.4, F.Cu at (170.9, 90.8)
- added C33: 10uF, Capacitor_SMD:CP_Elec_4x4.5, F.Cu at (134.0, 95.8)
- added C34: 0.1uF, Capacitor_SMD:C_1210_3225Metric_Pad1.33x2.70mm_HandSolder, F.Cu at (179.1, 83.2)
- added C35: 0.1uF, Capacitor_SMD:C_1210_3225Metric_Pad1.33x2.70mm_HandSolder, F.Cu at (179.1, 88.3)
- added C36: 3.3nF, Capacitor_SMD:C_0805_2012Metric_Pad1.18x1.45mm_HandSolder, F.Cu at (163.3, 92.7)
- added C37: 3.3nF, Capacitor_SMD:C_0805_2012Metric_Pad1.18x1.45mm_HandSolder, F.Cu at (140.3, 98.4)
- added C8: 1uF, Capacitor_SMD:CP_Elec_4x4.5, F.Cu at (128.3, 95.9)
- added J12: Conn_01x01_Female, Connector_Pin:Pin_D0.7mm_L6.5mm_W1.8mm_FlatFork, F.Cu at (180.0, 74.9)
- added J13: Conn_01x01_Female, Connector_Pin:Pin_D0.7mm_L6.5mm_W1.8mm_FlatFork, F.Cu at (184.8, 71.1)
- added R38: 12k, Resistor_SMD:R_0603_1608Metric_Pad0.98x0.95mm_HandSolder, F.Cu at (130.5, 89.5)
- added R39: 12k, Resistor_SMD:R_0603_1608Metric_Pad0.98x0.95mm_HandSolder, F.Cu at (123.5, 88.3)
- added R40: 1M, Resistor_SMD:R_0603_1608Metric_Pad0.98x0.95mm_HandSolder, F.Cu at (129.9, 80.6)
- added R41: 2k2, Resistor_SMD:R_0603_1608Metric_Pad0.98x0.95mm_HandSolder, F.Cu at (137.8, 88.3)
- added R42: 4k7, Resistor_SMD:R_0603_1608Metric_Pad0.98x0.95mm_HandSolder, F.Cu at (136.5, 85.4)
- added R43: 47k, Resistor_SMD:R_0603_1608Metric_Pad0.98x0.95mm_HandSolder, F.Cu at (190.8, 79.4)
- added R44: 2k2, Resistor_SMD:R_0603_1608Metric_Pad0.98x0.95mm_HandSolder, F.Cu at (166.1, 96.5)
- added R45: 2k2, Resistor_SMD:R_0603_1608Metric_Pad0.98x0.95mm_HandSolder, F.Cu at (166.4, 75.6)
- added R46: 10k, Resistor_SMD:R_0603_1608Metric_Pad0.98x0.95mm_HandSolder, F.Cu at (161.3, 100.3)
- added R47: 10k, Resistor_SMD:R_0603_1608Metric_Pad0.98x0.95mm_HandSolder, F.Cu at (138.1, 102.2)
- added R48: 470, Resistor_SMD:R_0603_1608Metric_Pad0.98x0.95mm_HandSolder, F.Cu at (161.6, 97.2)
- added R49: 470, Resistor_SMD:R_0603_1608Metric_Pad0.98x0.95mm_HandSolder, F.Cu at (143.5, 101.6)
- added RV2: 10k, Connector_PinHeader_2.54mm:PinHeader_1x03_P2.54mm_Vertical, F.Cu at (121.9, 78.1)
- added U11: CS4270-CZZ, Package_SO:TSSOP-24_4.4x7.8mm_P0.65mm, F.Cu at (170.8, 82.7)
- added U9: TL072, Package_SO:SOIC-8_3.9x4.9mm_P1.27mm, F.Cu at (130.1, 85.7)
- added X1: SG-5032CAN, Oscillator:Oscillator_SMD_SeikoEpson_SG8002CA-4Pin_7.0x5.0mm_HandSoldering, F.Cu at (171.5, 67.4)
- J4: value I2C Bus -> Conn_01x02_Pin; footprint Connector_PinHeader_2.54mm:PinHeader_1x03_P2.54mm_Vertical -> Connector_PinHeader_2.54mm:PinHeader_1x02_P2.54mm_Vertical
- moved J4 69.4 mm to (142.2, 77.5)
- moved H1 34.4 mm to (146.7, 52.1)
- moved D7 32.3 mm to (99.7, 86.4), turned to 180 degrees
- moved U6 29.8 mm to (37.5, 85.7)
- moved D5 28.4 mm to (95.9, 86.4), turned to 180 degrees
- moved D2 26.0 mm to (87.6, 86.4), turned to 180 degrees
- moved J5 24.8 mm to (72.4, 82.5)
- moved D3 23.3 mm to (79.4, 86.4), turned to 180 degrees
- moved R8 22.5 mm to (99.7, 78.7), turned to 90 degrees
- moved D6 22.5 mm to (83.2, 86.4), turned to 180 degrees
- moved D4 21.6 mm to (91.4, 86.4), turned to 180 degrees
- moved SW2 21.0 mm to (59.1, 84.5)
- moved U5 21.0 mm to (62.2, 75.6)
- moved SW1 21.0 mm to (54.6, 84.5)
- moved SW3 21.0 mm to (63.5, 84.5)
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Connections:
- C7 pad 2: Net-(J6-Pin_1) -> /Analog Preamp/Mic
- J4 pad 1: Net-(J4-Pin_1) -> GND
- R19 pad 1: Net-(J6-Pin_4) -> /Analog Preamp/DacR
- R20 pad 1: Net-(J3-Pin_1) -> Net-(C21-Pad1)
- R22 pad 1: Net-(J6-Pin_3) -> /Analog Preamp/DacL
- R23 pad 1: Net-(J3-Pin_2) -> Net-(C22-Pad1)
- U5 pad 27: Net-(J4-Pin_1) -> /Codec/SDA
- U5 pad 28: Net-(J4-Pin_2) -> /Codec/SCL
- U6 pad 5: Net-(J4-Pin_1) -> /Codec/SDA
- U6 pad 6: Net-(J4-Pin_2) -> /Codec/SCL
Routing:
- net Net-(U5-PD1): track 3.32 -> 44.8 mm
- net 3V3: track 67.0 -> 27.8 mm
- net Net-(J6-Pin_1): track 35.9 -> 0.00 mm
- net Net-(U5-PD0): track 4.58 -> 39.3 mm
- net Net-(J4-Pin_1): track 25.7 -> 0.00 mm, vias 2 -> 0
- net Net-(J4-Pin_2): track 24.5 -> 0.00 mm, vias 2 -> 0
- net Net-(U5-PC2): track 3.22 -> 25.3 mm
- net Net-(U5-PC3): track 9.52 -> 31.3 mm
- net Net-(J6-Pin_3): track 15.4 -> 0.00 mm
- net Net-(U5-PC1): track 5.15 -> 18.8 mm
- net Net-(C22-Pad1): track 0.00 -> 12.1 mm
- net /Codec/SCL: track 0.00 -> 11.6 mm
- net /Codec/SDA: track 0.00 -> 11.6 mm
- net Net-(J5-Pin_5): track 25.5 -> 14.2 mm, vias 3 -> 2
- net GND: track 89.0 -> 98.8 mm
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Other:
- board text added: "LED1"
- board text added: "LED2"
- board text added: "LED3"
