File: schematics/mic_extension_board/mic_extension_board.kicad_pcb (KiCad board)
At the start: 2 copper layers, 128.3 x 74.9 mm, 146 parts, among them J1 XLR3, J12 Conn_01x01_Female, J13 Conn_01x01_Female, J2 Conn_01x02_Male, J3 Aux In, J4 Conn_01x02_Pin, J5 Conn_02x03_Odd_Even, J6 Conn_01x03_Female, J7 XLR3, J8 XLR3, J9 Conn_01x03, P0 25k, P1 25k, P2 25k, SW1 Stompbutton 1, SW2 Stompbutton 2, SW3 Stompbutton 3, SW4 Enter, SW5 Exit, U1 TL074, U10 LM4881M/NOPB, U11 CS4270-CZZ, U12 128X64 OLED Display, U13 Debug Port, U14 AP63203WU, U2 Pico, U4 NE5534, U5 ATmega88A-A, U6 24LC128, U7 MC78M05_TO252, U8 MC78M05_TO252, U9 TL074, X1 SG-5032CAN

Commit message: pcb: layout changes, c headers: documentation
Parts:
- removed U8: MC78M05_TO252, Package_TO_SOT_SMD:TO-252-2
- added D10: SM6T12A, Diode_SMD:D_SMB, F.Cu at (78.3, 71.1)
- added D11: SM6T12A, Diode_SMD:D_SMB, F.Cu at (86.0, 71.1)
- added D9: SM6T12A, Diode_SMD:D_SMB, F.Cu at (97.8, 70.5)
- added U3: LM1117DT-5.0, Package_TO_SOT_SMD:TO-252-3_TabPin2, F.Cu at (90.2, 98.4)
- moved J2 32.1 mm to (76.7, 122.4)
- moved C14 16.9 mm to (81.8, 94.6)
- moved L1 10.4 mm to (88.0, 125.7)
- moved U14 10.4 mm to (86.7, 130.8)
- moved C40 10.4 mm to (93.0, 129.5)
- moved C5 10.2 mm to (82.5, 120.7)
- moved C6 10.2 mm to (82.5, 114.3)
- moved U7 9.76 mm to (80.0, 102.9)
- moved R41 9.38 mm to (95.2, 95.2), turned to -90 degrees
- moved C18 7.08 mm to (96.5, 90.2)
- moved TP2 7.00 mm to (76.2, 78.2)
- moved R42 6.71 mm to (99.1, 90.2)
- moved R3 6.34 mm to (78.7, 76.3)
- moved C2 5.58 mm to (92.6, 109.8)
- moved R44 5.58 mm to (88.7, 114.3)
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Routing:
- net GND: track 254.9 -> 236.4 mm, vias 29 -> 38
- net 5V: track 81.3 -> 99.2 mm
- net +9V: track 95.5 -> 111.1 mm
- net Net-(U1D-+): track 11.1 -> 23.4 mm
- net Net-(C4-Pad2): track 29.1 -> 40.4 mm, vias 2 -> 0
- net Net-(U1A--): track 30.4 -> 37.8 mm
- net Net-(D10-A1): track 3.59 -> 10.5 mm
- net Net-(D11-A1): track 4.49 -> 10.9 mm
- net /Codec/SDA: track 115.0 -> 120.5 mm
- net Net-(C20-Pad2): track 5.72 -> 11.2 mm
- net /Codec/SCL: track 116.9 -> 122.3 mm
- net Net-(U5-PB2): track 4.57 -> 9.91 mm
- net Net-(U5-PB1): track 6.12 -> 10.8 mm
- net VGND: track 82.3 -> 79.0 mm
- net Vin: track 40.8 -> 38.0 mm
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- added copper zone on B.Cu, net (none)
- added copper zone on In1.Cu, net GND
- removed copper zone on B.Cu, net GND
Other:
- copper layers 2 -> 4
- board text added: "128x64 OLED"
- board text added: "3V3"
- board text added: "CS"
- board text added: "DC"
- board text added: "Data"
- board text added: "GND"
- board text added: "RST"
- board text added: "SCK"

Commit message: fixed layout error, added copper fill
Connections:
- C17 pad 1: /Analog Preamp/Left Analog Out -> Net-(C17-Pad1)
- C17 pad 2: Net-(C17-Pad2) -> /Analog Preamp/Left Analog Out
- R24 pad 2: /Analog Preamp/Left Analog Out -> Net-(C17-Pad1)
- R25 pad 1: /Analog Preamp/Left Analog Out -> Net-(C17-Pad1)
- R33 pad 1: Net-(C17-Pad2) -> /Analog Preamp/Left Analog Out
- U9 pad 1: /Analog Preamp/Left Analog Out -> Net-(C17-Pad1)
Routing:
- net Net-(C17-Pad1): track 0.00 -> 37.7 mm
- net /Analog Preamp/Left Analog Out: track 43.9 -> 15.8 mm, vias 0 -> 2
- net Net-(C17-Pad2): track 3.29 -> 0.00 mm
Other:
- board text added: "Encoder"
- board text added: "Enter"
- board text added: "Exit"
- board text added: "RX"
- board text added: "SWCLK"
- board text added: "SWDIO"
- board text added: "TX"

Commit message: added decoupling caps at mic input
Parts:
- removed D10, D11: SM6T12A, Diode_SMD:D_SMB
- added C41: 10uF, Capacitor_SMD:CP_Elec_4x4.5, F.Cu at (85.1, 71.6)
- added C42: 10uF, Capacitor_SMD:CP_Elec_4x4.5, F.Cu at (76.7, 71.6)
Connections:
- J1 pad 2: Net-(D11-A1) -> Net-(C41-Pad2)
- J1 pad 3: Net-(D10-A1) -> Net-(C42-Pad2)
- R2 pad 1: Net-(D11-A1) -> Net-(C41-Pad1)
- R3 pad 1: Net-(D10-A1) -> Net-(C42-Pad1)
Routing:
- net Net-(D11-A1): track 10.9 -> 0.00 mm
- net Net-(D10-A1): track 10.5 -> 0.00 mm
- net Net-(C41-Pad2): track 0.00 -> 7.52 mm
- net GND: track 236.4 -> 229.8 mm, vias 38 -> 36
- net Net-(C41-Pad1): track 0.00 -> 4.39 mm
- net Net-(C42-Pad2): track 0.00 -> 3.67 mm
- net Net-(C42-Pad1): track 0.00 -> 2.85 mm
- net Net-(C17-Pad1): track 37.7 -> 37.2 mm
