File: schematics/mic_extension_board/uicontroller.kicad_sch (KiCad schematic)
At the start: 20 parts, among them J4 I2C Bus, J5 6Pin ISP, SW1 Stompbutton 1, SW2 Stompbutton 2, SW3 Stompbutton 3, U5 ATmega88A-A, U6 24LC128

Commit message: more layouting
Parts:
- removed J4: I2C Bus, Connector_PinHeader_2.54mm:PinHeader_1x03_P2.54mm_Vertical, symbol Connector:Conn_01x03_Female
Connections:
- net SDA: now reaches U5.27 (PC4), U6.5 (SDA)
- net SCL: now reaches U5.28 (PC5), U6.6 (SCL)
Changed lines of the file:
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@@
   (junction (at 91.44 78.74) (diameter 0) (color 0 0 0 0)
-  )
-  (junction (at 102.87 67.31) (diameter 0) (color 0 0 0 0)
   )
   (junction (at 109.22 59.69) (diameter 0) (color 0 0 0 0)
@@
     (stroke (width 0) (type default))
   )
-  (wire (pts (xy 102.87 67.31) (xy 118.11 67.31))
-    (stroke (width 0) (type default))
-  )
   (wire (pts (xy 138.43 71.12) (xy 138.43 120.65))
     (stroke (width 0) (type default))
@@
     (stroke (width 0) (type default))
   )
-  (wire (pts (xy 111.76 57.15) (xy 118.11 57.15))
-    (stroke (width 0) (type default))
-  )
-  (wire (pts (xy 109.22 59.69) (xy 118.11 59.69))
+  (wire (pts (xy 111.76 57.15) (xy 114.3 57.15))
+    (stroke (width 0) (type default))
+  )
+  (wire (pts (xy 109.22 59.69) (xy 114.3 59.69))
     (stroke (width 0) (type default))
   )
@@
     (stroke (width 0) (type default))
   )
-  (wire (pts (xy 118.11 67.31) (xy 118.11 62.23))
-    (stroke (width 0) (type default))
-  )
   (wire (pts (xy 166.37 102.87) (xy 175.26 102.87))
     (stroke (width 0) (type default))
@@
     (stroke (width 0) (type default))
   )
-  (wire (pts (xy 102.87 68.58) (xy 102.87 67.31))
-    (stroke (width 0) (type default))
-  )
   (wire (pts (xy 137.16 118.11) (xy 137.16 72.39))
     (stroke (width 0) (type default))
@@
     (stroke (width 0) (type default))
   )
-  (wire (pts (xy 102.87 62.23) (xy 102.87 67.31))
+  (wire (pts (xy 102.87 62.23) (xy 102.87 68.58))
     (stroke (width 0) (type default))
   )
@@
       (effects (font (size 1.27 1.27)) (justify left) hide)
     )
+  )
+  (hierarchical_label "SCL" (shape input) (at 114.3 59.69 0) (fields_autoplaced)
+    (effects (font (size 1.27 1.27)) (justify left))
+  )
+  (hierarchical_label "SDA" (shape input) (at 114.3 57.15 0) (fields_autoplaced)
+    (effects (font (size 1.27 1.27)) (justify left))
   )
   (symbol (lib_id "power:GND") (at 149.86 102.87 0) (unit 1)
@@
         )
       )
-    )
-  )
-  (symbol (lib_id "Connector:Conn_01x03_Female") (at 123.19 59.69 0) (unit 1)
-    (in_bom yes) (on_board yes) (dnp no) (fields_autoplaced)
-    (property "Reference" "J4" (at 123.9012 58.8553 0)
-      (effects (font (size 1.27 1.27)) (justify left))
-    )
-    (property "Value" "I2C Bus" (at 123.9012 61.3922 0)
-      (effects (font (size 1.27 1.27)) (justify left))
-    )
-    (property "Footprint" "Connector_PinHeader_2.54mm:PinHeader_1x03_P2.54mm_Vertical" (at 123.19 59.69 0)
-      (effects (font (size 1.27 1.27)) hide)
-    )
-    (property "Datasheet" "~" (at 123.19 59.69 0)
-      (effects (font (size 1.27 1.27)) hide)
-    )
-    (pin "1")
-    (pin "2")
-    (pin "3")
-    (instances
-      (project "mic_extension_board"
-        (path "/e63e39d7-6ac0-4ffd-8aa3-1841a4541b55"
-          (reference "J4") (unit 1)
-        )
-        (path "/e63e39d7-6ac0-4ffd-8aa3-1841a4541b55/f9ef1368-05a5-440b-8b6f-d12c6284b642"
-          (reference "J4") (unit 1)
-        )
-      )

Commit message: finished full board
Parts:
- J5: value 6Pin ISP -> Conn_02x03_Odd_Even
- R11, R12, R13, R14, R7, R8: value 180 -> R
- R9: value 10k -> R
- SW1: value Stompbutton 1 -> SW_Push
- SW2: value Stompbutton 2 -> SW_Push
- SW3: value Stompbutton 3 -> SW_Push
Changed lines of the file:
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@@
       (effects (font (size 1.27 1.27)))
     )
-    (property "Value" "Stompbutton 1" (at 144.78 77.1961 0)
+    (property "Value" "SW_Push" (at 144.78 77.1961 0)
       (effects (font (size 1.27 1.27)))
     )
@@
       (effects (font (size 1.27 1.27)) (justify left))
     )
-    (property "Value" "180" (at 123.19 118.11 90)
+    (property "Value" "R" (at 123.19 118.11 90)
       (effects (font (size 1.27 1.27)) (justify left))
     )
@@
       (effects (font (size 1.27 1.27)) (justify left))
     )
-    (property "Value" "180" (at 123.19 113.03 90)
+    (property "Value" "R" (at 123.19 113.03 90)
       (effects (font (size 1.27 1.27)) (justify left))
     )
@@
       (effects (font (size 1.27 1.27)) (justify left))
     )
-    (property "Value" "180" (at 123.19 115.57 90)
+    (property "Value" "R" (at 123.19 115.57 90)
       (effects (font (size 1.27 1.27)) (justify left))
     )
@@
       (effects (font (size 1.27 1.27)) (justify left))
     )
-    (property "Value" "180" (at 110.49 135.89 90)
+    (property "Value" "R" (at 110.49 135.89 90)
       (effects (font (size 1.27 1.27)) (justify left))
     )
@@
       (effects (font (size 1.27 1.27)) (justify left))
     )
-    (property "Value" "180" (at 110.49 133.35 90)
+    (property "Value" "R" (at 110.49 133.35 90)
       (effects (font (size 1.27 1.27)) (justify left))
     )
@@
       (effects (font (size 1.27 1.27)))
     )
-    (property "Value" "Stompbutton 2" (at 144.78 86.0861 0)
+    (property "Value" "SW_Push" (at 144.78 86.0861 0)
       (effects (font (size 1.27 1.27)))
     )
@@
       (effects (font (size 1.27 1.27)) (justify left))
     )
-    (property "Value" "10k" (at 109.22 109.22 0)
+    (property "Value" "R" (at 109.22 109.22 0)
       (effects (font (size 1.27 1.27)) (justify left))
     )
@@
       (effects (font (size 1.27 1.27)))
     )
-    (property "Value" "6Pin ISP" (at 133.35 134.7271 0)
+    (property "Value" "Conn_02x03_Odd_Even" (at 133.35 134.7271 0)
       (effects (font (size 1.27 1.27)))
     )
@@
       (effects (font (size 1.27 1.27)))
     )
-    (property "Value" "Stompbutton 3" (at 144.78 94.9761 0)
+    (property "Value" "SW_Push" (at 144.78 94.9761 0)
       (effects (font (size 1.27 1.27)))
     )
@@
       (effects (font (size 1.27 1.27)) (justify left))
     )
-    (property "Value" "180" (at 123.19 120.65 90)
-      (effects (font (size 1.27 1.27)) (justify left))
-    )
+    (property "Value" "R" (at 123.19 120.65 90)
+      (effects (font (size 1.27 1.27)) (justify left))
+    )

Commit message: re-added component values previously lost due to kicad mishap
Parts:
- R11, R12, R13, R14, R7, R8: value R -> 180
- R9: value R -> 10k
- SW1: value SW_Push -> Stompbutton 1
- SW2: value SW_Push -> Stompbutton 2
- SW3: value SW_Push -> Stompbutton 3
Changed lines of the file:
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@@
       (effects (font (size 1.27 1.27)))
     )
-    (property "Value" "SW_Push" (at 144.78 77.1961 0)
+    (property "Value" "Stompbutton 1" (at 144.78 77.1961 0)
       (effects (font (size 1.27 1.27)))
     )
@@
       (effects (font (size 1.27 1.27)) (justify left))
     )
-    (property "Value" "R" (at 123.19 118.11 90)
+    (property "Value" "180" (at 123.19 118.11 90)
       (effects (font (size 1.27 1.27)) (justify left))
     )
@@
       (effects (font (size 1.27 1.27)) (justify left))
     )
-    (property "Value" "R" (at 123.19 113.03 90)
+    (property "Value" "180" (at 123.19 113.03 90)
       (effects (font (size 1.27 1.27)) (justify left))
     )
@@
       (effects (font (size 1.27 1.27)) (justify left))
     )
-    (property "Value" "R" (at 123.19 115.57 90)
+    (property "Value" "180" (at 123.19 115.57 90)
       (effects (font (size 1.27 1.27)) (justify left))
     )
@@
       (effects (font (size 1.27 1.27)) (justify left))
     )
-    (property "Value" "R" (at 110.49 135.89 90)
+    (property "Value" "180" (at 110.49 135.89 90)
       (effects (font (size 1.27 1.27)) (justify left))
     )
@@
       (effects (font (size 1.27 1.27)) (justify left))
     )
-    (property "Value" "R" (at 110.49 133.35 90)
+    (property "Value" "180" (at 110.49 133.35 90)
       (effects (font (size 1.27 1.27)) (justify left))
     )
@@
       (effects (font (size 1.27 1.27)))
     )
-    (property "Value" "SW_Push" (at 144.78 86.0861 0)
+    (property "Value" "Stompbutton 2" (at 144.78 86.0861 0)
       (effects (font (size 1.27 1.27)))
     )
@@
       (effects (font (size 1.27 1.27)) (justify left))
     )
-    (property "Value" "R" (at 109.22 109.22 0)
+    (property "Value" "10k" (at 109.22 109.22 0)
       (effects (font (size 1.27 1.27)) (justify left))
     )
@@
       (effects (font (size 1.27 1.27)))
     )
-    (property "Value" "SW_Push" (at 144.78 94.9761 0)
+    (property "Value" "Stompbutton 3" (at 144.78 94.9761 0)
       (effects (font (size 1.27 1.27)))
     )
@@
       (effects (font (size 1.27 1.27)) (justify left))
     )
-    (property "Value" "R" (at 123.19 120.65 90)
-      (effects (font (size 1.27 1.27)) (justify left))
-    )
+    (property "Value" "180" (at 123.19 120.65 90)
+      (effects (font (size 1.27 1.27)) (justify left))
+    )
