File: schematics/mic_extension_board/analogpreamp.kicad_sch (KiCad schematic)
At the start: 45 parts, among them J1 XLR3, J3 Aux In, J6 Input/Output, J7 XLR3, J8 XLR3, U1 TL074, U2 TL072, U4 NE5534

Commit message: more layouting
Parts:
- removed J6: Input/Output, Connector_PinHeader_2.54mm:PinHeader_1x04_P2.54mm_Vertical, symbol Connector:Conn_01x04_Female
- added C10, C21, C22: 4.7uF, Capacitor_SMD:CP_Elec_4x4.5, symbol Device:C_Polarized
- added C18: 220pF, Capacitor_SMD:C_0603_1608Metric_Pad1.08x0.95mm_HandSolder, symbol Device:C
- added C19, C20, C8: 1uF, Capacitor_SMD:CP_Elec_4x4.5, symbol Device:C_Polarized
- added J4: Conn_01x02_Pin, Connector_PinHeader_2.54mm:PinHeader_1x02_P2.54mm_Vertical, symbol Connector:Conn_01x02_Pin
- added R38, R39: 12k, Resistor_SMD:R_0603_1608Metric_Pad0.98x0.95mm_HandSolder, symbol Device:R
- added R40: 1M, Resistor_SMD:R_0603_1608Metric_Pad0.98x0.95mm_HandSolder, symbol Device:R
- added R41: 2k2, Resistor_SMD:R_0603_1608Metric_Pad0.98x0.95mm_HandSolder, symbol Device:R
- added R42: 4k7, Resistor_SMD:R_0603_1608Metric_Pad0.98x0.95mm_HandSolder, symbol Device:R
- added RV2: 10k, Connector_PinHeader_2.54mm:PinHeader_1x03_P2.54mm_Vertical, symbol Device:R_Potentiometer
- added U9: TL072, Package_SO:SOIC-8_3.9x4.9mm_P1.27mm, symbol Amplifier_Operational:TL072
Connections:
- net +9V: now also R38.1, U9.8 (V+)
- net GND: now also C10.2, C8.2, J4.1 (Pin_1), R39.2, RV2.3, U9.4 (V-)
- net at R20.1: now also C21.1; no longer J3.1 (Pin_1)
- net Mic: now reaches C7.2
- net DacL: now reaches R22.1
- net DacR: now reaches R19.1
- net at R23.1: now also C22.1; no longer J3.2 (Pin_2)
- new net: C21.2, J3.1 (Pin_1)
- new net: C19.1, R40.2, U9.5 (+)
- new net: C18.1, R41.1, R42.1, U9.6 (-)
- new net: C18.2, C20.1, R42.2, U9.7
- new net: R40.1, U9.1, U9.2 (-)
- new net: C8.1, R38.2, R39.1, U9.3 (+)
- new net: C20.2, RV2.1
- new net: C10.1, R41.2
- new net: C22.2, J3.2 (Pin_2)
- new net: C19.2, J4.2 (Pin_2)
- new net HiZ: RV2.2

Commit message: finished full board
Parts:
- removed U2, U9: TL072, Package_SO:SOIC-8_3.9x4.9mm_P1.27mm, symbol Amplifier_Operational:TL072
- added U9: TL074, Package_SO:SOIC-14_3.9x8.7mm_P1.27mm, symbol Amplifier_Operational:TL074
- C1: value 33pF -> C; footprint Capacitor_SMD:C_0603_1608Metric_Pad1.08x0.95mm_HandSolder -> Capacitor_SMD:C_0805_2012Metric_Pad1.18x1.45mm_HandSolder
- C10, C21, C22: value 4.7uF -> C_Polarized
- C13, C15, C17, C3: value 10uF -> C_Polarized
- C16: value 0.1uF -> C
- C18: value 220pF -> C
- C19, C20, C7, C8: value 1uF -> C_Polarized
- C4: value 47pF -> C
- R1, R2, R3, R4: value 22k -> R
- R10, R19, R21, R22, R24, R25, R26, R27, R28, R31, R34, R35: value 10k -> R
- R20, R23, R42, R5: value 4k7 -> R
- R30, R32, R33, R6: value 150 -> R
- R36, R37, R38, R39: value 12k -> R
- R40: value 1M -> R
- R41: value 2k2 -> R
- RV1: value 100k -> R_Potentiometer
- RV2: value 10k -> R_Potentiometer
Connections:
- net +9V: now also U9.4 (V+)
- net GND: now also U1.10 (+), U9.11 (V-)
- net Left Analog Out: now also U9.1
- net VGND: now also U1.13 (-), U1.14, U9.10 (+), U9.12 (+), U9.3 (+), U9.5 (+); no longer U1.10 (+), U1.12 (+), U1.6 (-), U1.7
- net at R21.2, R27.1: now also U9.9 (-); no longer U1.9 (-)
- net at C13.1, R27.2: now also U9.8; no longer U1.8
- net at R19.2, R20.2, R26.1: now also U9.13 (-); no longer U1.13 (-)
- net at C16.1, R36.2, R37.1: now also U1.12 (+); no longer U1.5 (+)
- net at R22.2, R23.2, R24.1: now also U9.2 (-)
- net at C19.1, R40.2: now also U1.5 (+)
- net at C18.1, R41.1, R42.1: now also U1.6 (-)
- net at C18.2, C20.1, R42.2: now also U1.7
- net at R40.1: now also C8.1, R38.2, R39.1
- net at R25.2, R28.1: now also U9.6 (-)
- net at C15.1, R28.2: now also U9.7
- net at C3.1, R21.1, R26.2: now also U9.14; no longer U1.14
- new net: U1.8, U1.9 (-)
Other:
- moved on the sheet: U1B, U1C, U1D

Commit message: re-added component values previously lost due to kicad mishap
Parts:
- C1: value C -> 33pF
- C10, C21, C22: value C_Polarized -> 4.7uF
- C13, C15, C17, C3: value C_Polarized -> 10uF
- C16: value C -> 0.1uF
- C18: value C -> 220pF
- C19, C20, C7, C8: value C_Polarized -> 1uF
- C4: value C -> 47pF
- R1, R2, R3, R4: value R -> 22k
- R10, R19, R21, R22, R24, R25, R26, R27, R28, R31, R34, R35: value R -> 10k
- R20, R23, R42, R5: value R -> 4k7
- R30, R32, R33, R6: value R -> 150
- R36, R37, R38, R39: value R -> 12k
- R40: value R -> 1M
- R41: value R -> 2k2
- RV1: value R_Potentiometer -> 100k
- RV2: value R_Potentiometer -> 10k

Commit message: pcb: layout changes, c headers: documentation
Parts:
- added D10, D11, D9: SM6T12A, Diode_SMD:D_SMB, symbol Diode:SM6T12A
Connections:
- net GND: now also D10.2 (A2), D11.2 (A2), D9.2 (A2)
- net at J1.2, R2.1: now also D11.1 (A1)
- net at J1.3, R3.1: now also D10.1 (A1)
- net at C19.2, J4.2 (Pin_2): now also D9.1 (A1)
Changed lines of the file:
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@@
 (kicad_sch (version 20230121) (generator eeschema)
   (paper "A4")
+  (junction (at 35.56 134.62) (diameter 0) (color 0 0 0 0)
+  )
   (junction (at 194.31 63.5) (diameter 0) (color 0 0 0 0)
   )
@@
   (junction (at 41.91 111.76) (diameter 0) (color 0 0 0 0)
   )
+  (junction (at 45.72 67.31) (diameter 0) (color 0 0 0 0)
+  )
   (junction (at 57.15 50.8) (diameter 0) (color 0 0 0 0)
   )
   (junction (at 118.11 111.76) (diameter 0) (color 0 0 0 0)
   )
+  (junction (at 50.8 62.23) (diameter 0) (color 0 0 0 0)
+  )
   (junction (at 95.25 69.85) (diameter 0) (color 0 0 0 0)
   )
@@
   (junction (at 90.17 69.85) (diameter 0) (color 0 0 0 0)
   )
+  (junction (at 46.99 74.93) (diameter 0) (color 0 0 0 0)
+  )
   (junction (at 86.36 101.6) (diameter 0) (color 0 0 0 0)
   )
@@
     (stroke (width 0) (type default))
   )
+  (wire (pts (xy 50.8 69.85) (xy 50.8 74.93))
+    (stroke (width 0) (type default))
+  )
   (wire (pts (xy 123.19 93.98) (xy 129.54 93.98))
     (stroke (width 0) (type default))
@@
     (stroke (width 0) (type default))
   )
-  (wire (pts (xy 161.29 45.72) (xy 161.29 38.1))
+  (wire (pts (xy 161.29 45.72) (xy 161.29 36.83))
     (stroke (width 0) (type default))
   )
@@
     (stroke (width 0) (type default))
   )
+  (wire (pts (xy 46.99 74.93) (xy 45.72 74.93))
+    (stroke (width 0) (type default))
+  )
   (wire (pts (xy 86.36 101.6) (xy 90.17 101.6))
     (stroke (width 0) (type default))
@@
     (stroke (width 0) (type default))
   )
+  (wire (pts (xy 45.72 67.31) (xy 50.8 67.31))
+    (stroke (width 0) (type default))
+  )
   (wire (pts (xy 217.17 55.88) (xy 217.17 64.77))
     (stroke (width 0) (type default))
   )
+  (wire (pts (xy 35.56 134.62) (xy 29.21 134.62))
+    (stroke (width 0) (type default))
+  )
   (wire (pts (xy 209.55 95.25) (xy 210.82 95.25))
     (stroke (width 0) (type default))
@@
     (stroke (width 0) (type default))
   )
-  (wire (pts (xy 43.18 67.31) (xy 50.8 67.31))
-    (stroke (width 0) (type default))
-  )
-  (wire (pts (xy 40.64 134.62) (xy 29.21 134.62))
+  (wire (pts (xy 43.18 67.31) (xy 45.72 67.31))
+    (stroke (width 0) (type default))
+  )
+  (wire (pts (xy 40.64 134.62) (xy 35.56 134.62))
     (stroke (width 0) (type default))
   )
@@
     (stroke (width 0) (type default))
   )
-  (wire (pts (xy 162.56 38.1) (xy 162.56 36.83))
-    (stroke (width 0) (type default))
-  )
   (wire (pts (xy 190.5 102.87) (xy 190.5 95.25))
     (stroke (width 0) (type default))
@@
     (stroke (width 0) (type default))
   )
-  (wire (pts (xy 161.29 38.1) (xy 162.56 38.1))
-    (stroke (width 0) (type default))
-  )
   (wire (pts (xy 90.17 69.85) (xy 90.17 64.77))
     (stroke (width 0) (type default))
@@
     (stroke (width 0) (type default))
   )
-  (wire (pts (xy 162.56 36.83) (xy 166.37 36.83))
+  (wire (pts (xy 161.29 36.83) (xy 166.37 36.83))
     (stroke (width 0) (type default))
   )
@@
   )
   (wire (pts (xy 106.68 69.85) (xy 106.68 62.23))
+    (stroke (width 0) (type default))
+  )
+  (wire (pts (xy 50.8 74.93) (xy 46.99 74.93))
     (stroke (width 0) (type default))
   )
@@
   (symbol (lib_id "Device:R") (at 54.61 62.23 90) (unit 1)
     (in_bom yes) (on_board yes) (dnp no)
-    (property "Reference" "R2" (at 50.8 64.77 90)
+    (property "Reference" "R2" (at 49.53 60.96 90)
       (effects (font (size 1.27 1.27)))
     )
@@
     )
   )
+  (symbol (lib_id "power:GND") (at 35.56 142.24 0) (unit 1)
+    (in_bom yes) (on_board yes) (dnp no) (fields_autoplaced)
+    (property "Reference" "#PWR0104" (at 35.56 148.59 0)
+      (effects (font (size 1.27 1.27)) hide)
+    )
+    (property "Value" "GND" (at 35.56 146.6834 0)
+      (effects (font (size 1.27 1.27)))
+    )
+    (property "Footprint" "" (at 35.56 142.24 0)
+      (effects (font (size 1.27 1.27)) hide)
+    )
+    (property "Datasheet" "" (at 35.56 142.24 0)
+      (effects (font (size 1.27 1.27)) hide)
+    )
+    (pin "1")
+    (instances
+      (project "mic_extension_board"
+        (path "/e63e39d7-6ac0-4ffd-8aa3-1841a4541b55"
+          (reference "#PWR0104") (unit 1)
+        )
+        (path "/e63e39d7-6ac0-4ffd-8aa3-1841a4541b55/9b4677b6-5618-4dd2-a345-e4ce8cf01c2f"
+          (reference "#PWR050") (unit 1)
+        )
+      )
+    )
+  )
   (symbol (lib_id "Device:R") (at 41.91 107.95 0) (unit 1)
     (in_bom yes) (on_board yes) (dnp no) (fields_autoplaced)
@@
     )
   )
+  (symbol (lib_id "Diode:SM6T12A") (at 35.56 138.43 270) (unit 1)
+    (in_bom yes) (on_board yes) (dnp no) (fields_autoplaced)
+    (property "Reference" "D9" (at 38.1 137.16 90)
+      (effects (font (size 1.27 1.27)) (justify left))
+    )
+    (property "Value" "SM6T12A" (at 38.1 139.7 90)
+      (effects (font (size 1.27 1.27)) (justify left))
+    )
+    (property "Footprint" "Diode_SMD:D_SMB" (at 30.48 138.43 0)
+      (effects (font (size 1.27 1.27)) hide)
+    )
+    (property "Datasheet" "https://www.st.com/resource/en/datasheet/sm6t.pdf" (at 35.56 137.16 0)
+      (effects (font (size 1.27 1.27)) hide)
+    )
+    (pin "2")
+    (pin "1")
+    (instances
+      (project "mic_extension_board"
+        (path "/e63e39d7-6ac0-4ffd-8aa3-1841a4541b55/9b4677b6-5618-4dd2-a345-e4ce8cf01c2f"
+          (reference "D9") (unit 1)
+        )
+      )
+    )
+  )
   (symbol (lib_id "power:GND") (at 54.61 100.33 0) (unit 1)
     (in_bom yes) (on_board yes) (dnp no) (fields_autoplaced)
@@
         (path "/e63e39d7-6ac0-4ffd-8aa3-1841a4541b55/9b4677b6-5618-4dd2-a345-e4ce8cf01c2f"
           (reference "#PWR017") (unit 1)
+        )
+      )
+    )
+  )
+  (symbol (lib_id "Diode:SM6T12A") (at 50.8 66.04 270) (unit 1)
+    (in_bom yes) (on_board yes) (dnp no)
+    (property "Reference" "D11" (at 45.72 63.5 90)
+      (effects (font (size 1.27 1.27)) (justify left))
+    )
+    (property "Value" "SM6T12A" (at 40.64 66.04 90)
+      (effects (font (size 1.27 1.27)) (justify left))
+    )
+    (property "Footprint" "Diode_SMD:D_SMB" (at 45.72 66.04 0)
+      (effects (font (size 1.27 1.27)) hide)
+    )
+    (property "Datasheet" "https://www.st.com/resource/en/datasheet/sm6t.pdf" (at 50.8 64.77 0)
+      (effects (font (size 1.27 1.27)) hide)
+    )
+    (pin "2")
+    (pin "1")
+    (instances
+      (project "mic_extension_board"
+        (path "/e63e39d7-6ac0-4ffd-8aa3-1841a4541b55/9b4677b6-5618-4dd2-a345-e4ce8cf01c2f"
+          (reference "D11") (unit 1)
         )
       )
@@
         (path "/e63e39d7-6ac0-4ffd-8aa3-1841a4541b55/9b4677b6-5618-4dd2-a345-e4ce8cf01c2f"
           (reference "U9") (unit 2)
+        )
+      )
+    )
+  )
+  (symbol (lib_id "power:GND") (at 46.99 74.93 0) (unit 1)
+    (in_bom yes) (on_board yes) (dnp no) (fields_autoplaced)
+    (property "Reference" "#PWR01" (at 46.99 81.28 0)
+      (effects (font (size 1.27 1.27)) hide)
+    )
+    (property "Value" "GND" (at 46.99 79.3734 0)
+      (effects (font (size 1.27 1.27)))
+    )
+    (property "Footprint" "" (at 46.99 74.93 0)
+      (effects (font (size 1.27 1.27)) hide)
+    )
+    (property "Datasheet" "" (at 46.99 74.93 0)
+      (effects (font (size 1.27 1.27)) hide)
+    )
+    (pin "1")
+    (instances
+      (project "mic_extension_board"
+        (path "/e63e39d7-6ac0-4ffd-8aa3-1841a4541b55"
+          (reference "#PWR01") (unit 1)
+        )
+        (path "/e63e39d7-6ac0-4ffd-8aa3-1841a4541b55/9b4677b6-5618-4dd2-a345-e4ce8cf01c2f"
+          (reference "#PWR051") (unit 1)
         )
       )
@@
     )
   )
+  (symbol (lib_id "Diode:SM6T12A") (at 45.72 71.12 270) (unit 1)
+    (in_bom yes) (on_board yes) (dnp no)
+    (property "Reference" "D10" (at 39.37 69.85 90)
+      (effects (font (size 1.27 1.27)) (justify left))
+    )
+    (property "Value" "SM6T12A" (at 34.29 72.39 90)
+      (effects (font (size 1.27 1.27)) (justify left))
+    )
+    (property "Footprint" "Diode_SMD:D_SMB" (at 40.64 71.12 0)
+      (effects (font (size 1.27 1.27)) hide)
+    )
+    (property "Datasheet" "https://www.st.com/resource/en/datasheet/sm6t.pdf" (at 45.72 69.85 0)
+      (effects (font (size 1.27 1.27)) hide)
+    )
+    (pin "2")
+    (pin "1")
+    (instances
+      (project "mic_extension_board"
+        (path "/e63e39d7-6ac0-4ffd-8aa3-1841a4541b55/9b4677b6-5618-4dd2-a345-e4ce8cf01c2f"
+          (reference "D10") (unit 1)
+        )
+      )
+    )
+  )
   (symbol (lib_id "power:GND") (at 35.56 59.69 0) (unit 1)
     (in_bom yes) (on_board yes) (dnp no) (fields_autoplaced)
@@
   (symbol (lib_id "Device:R") (at 54.61 67.31 90) (unit 1)
     (in_bom yes) (on_board yes) (dnp no)
-    (property "Reference" "R3" (at 50.8 69.85 90)
-      (effects (font (size 1.27 1.27)))
-    )
+    (property "Reference" "R3" (at 58.42 64.77 90)
+      (effects (font (size 1.27 1.27)))
+    )

Commit message: fixed layout error, added copper fill
Connections:
- net Left Analog Out: now also C17.2, R33.1; no longer C17.1, R24.2, R25.1, U9.1
- new net: C17.1, R24.2, R25.1, U9.1
