File: schematics/mic_extension_board/mic_extension_board.kicad_sch (KiCad schematic)
At the start: 75 parts, among them J1 XLR3, J10 Conn_01x01_Male, J2 Conn_01x02_Male, J3 Aux In, J4 I2C Bus, J5 6Pin ISP, J6 Input/Output, J7 XLR3, J8 XLR3, J9 Conn_01x03_Female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

Commit message: schematics changed and added gitignore files
Parts:
- U10: symbol 2023-02-24_23-31-36:LM4881M/NOPB -> 2023-02-24_23-31-36:LM4881M/NOPB
