File: schematics/full_board_pico_seed/codec.kicad_sch (KiCad schematic)
At the start: 18 parts, among them U5 PCM3060, X1 SG-5032CAN 12.288MHz

Commit message: schematic change
Parts:
- removed C10, C12: 10uF, Capacitor_SMD:CP_Elec_4x4.5, symbol Device:C_Polarized
- renumbered C28 to C26, C5 to C7, TP7 to TP10, TP5 to TP4, TP4 to TP5, TP8 to TP7, TP9 to TP8, TP10 to TP9
Connections:
- net codec_in_a: now also U5.25 (V_{IN}L)
- net codec_in_b: now also U5.26 (V_{IN}R)
Changed lines of the file:
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@@
 	(wire
 		(pts
-			(xy 144.78 66.04) (xy 153.67 66.04)
+			(xy 144.78 66.04) (xy 170.18 66.04)
 		)
 		(stroke
@@
 	(wire
 		(pts
-			(xy 161.29 63.5) (xy 170.18 63.5)
-		)
-		(stroke
-			(width 0)
-			(type default)
-		)
-	)
-	(wire
-		(pts
 			(xy 129.54 33.02) (xy 170.18 33.02)
 		)
@@
 	(wire
 		(pts
-			(xy 170.18 66.04) (xy 161.29 66.04)
-		)
-		(stroke
-			(width 0)
-			(type default)
-		)
-	)
-	(wire
-		(pts
 			(xy 170.18 86.36) (xy 163.83 86.36)
 		)
@@
 	(wire
 		(pts
-			(xy 142.24 58.42) (xy 142.24 121.92)
+			(xy 142.24 63.5) (xy 142.24 121.92)
 		)
 		(stroke
@@
 	(wire
 		(pts
-			(xy 142.24 58.42) (xy 153.67 58.42)
+			(xy 142.24 63.5) (xy 170.18 63.5)
 		)
 		(stroke
@@
 		(pts
 			(xy 97.79 33.02) (xy 97.79 39.37)
-		)
-		(stroke
-			(width 0)
-			(type default)
-		)
-	)
-	(wire
-		(pts
-			(xy 161.29 58.42) (xy 161.29 63.5)
 		)
 		(stroke
@@
 		(dnp no)
 		(fields_autoplaced yes)
-		(property "Reference" "TP8"
+		(property "Reference" "TP7"
 			(at 153.67 76.708 0)
 			(effects
@@
 			(project "full_board_pico_seed"
 				(path "/e63e39d7-6ac0-4ffd-8aa3-1841a4541b55/6ec17984-49ce-45c2-b1f4-ed6e904b8c80"
-					(reference "TP8")
+					(reference "TP7")
 					(unit 1)
 				)
@@
 		(on_board yes)
 		(dnp no)
-		(property "Reference" "TP5"
+		(property "Reference" "TP4"
 			(at 203.2 75.184 90)
 			(effects
@@
 			(project "full_board_pico_seed"
 				(path "/e63e39d7-6ac0-4ffd-8aa3-1841a4541b55/6ec17984-49ce-45c2-b1f4-ed6e904b8c80"
-					(reference "TP5")
+					(reference "TP4")
 					(unit 1)
 				)
@@
 		(on_board yes)
 		(dnp no)
-		(property "Reference" "TP9"
+		(property "Reference" "TP8"
 			(at 130.81 96.52 0)
 			(effects
@@
 			(project "full_board_pico_seed"
 				(path "/e63e39d7-6ac0-4ffd-8aa3-1841a4541b55/6ec17984-49ce-45c2-b1f4-ed6e904b8c80"
-					(reference "TP9")
+					(reference "TP8")
 					(unit 1)
 				)
@@
 		(on_board yes)
 		(dnp no)
-		(property "Reference" "C28"
+		(property "Reference" "C26"
 			(at 222.758 83.312 0)
 			(effects
@@
 			(project "full_board_pico_seed"
 				(path "/e63e39d7-6ac0-4ffd-8aa3-1841a4541b55/6ec17984-49ce-45c2-b1f4-ed6e904b8c80"
-					(reference "C28")
+					(reference "C26")
 					(unit 1)
 				)
@@
 		(on_board yes)
 		(dnp no)
-		(property "Reference" "TP10"
+		(property "Reference" "TP9"
 			(at 113.03 74.93 0)
 			(effects
@@
 			(project "full_board_pico_seed"
 				(path "/e63e39d7-6ac0-4ffd-8aa3-1841a4541b55/6ec17984-49ce-45c2-b1f4-ed6e904b8c80"
-					(reference "TP10")
+					(reference "TP9")
 					(unit 1)
 				)
@@
 		(on_board yes)
 		(dnp no)
-		(property "Reference" "TP7"
+		(property "Reference" "TP10"
 			(at 157.48 87.63 0)
 			(effects
@@
 			(project "full_board_pico_seed"
 				(path "/e63e39d7-6ac0-4ffd-8aa3-1841a4541b55/6ec17984-49ce-45c2-b1f4-ed6e904b8c80"
-					(reference "TP7")
+					(reference "TP10")
 					(unit 1)
 				)
@@
 			(project "full_board_pico_seed"
 				(path "/e63e39d7-6ac0-4ffd-8aa3-1841a4541b55/6ec17984-49ce-45c2-b1f4-ed6e904b8c80"
-					(reference "R33")
-					(unit 1)
-				)
-			)
-		)
-	)
-	(symbol
-		(lib_id "Device:C_Polarized")
-		(at 157.48 66.04 270)
-		(unit 1)
-		(exclude_from_sim no)
-		(in_bom yes)
-		(on_board yes)
-		(dnp no)
-		(property "Reference" "C12"
-			(at 152.146 69.342 90)
-			(effects
-				(font
-					(size 1.27 1.27)
-				)
-			)
-		)
-		(property "Value" "10uF"
-			(at 152.4 67.31 90)
-			(effects
-				(font
-					(size 1.27 1.27)
-				)
-			)
-		)
-		(property "Footprint" "Capacitor_SMD:CP_Elec_4x4.5"
-			(at 153.67 67.0052 0)
-			(effects
-				(font
-					(size 1.27 1.27)
-				)
-				(hide yes)
-			)
-		)
-		(property "Datasheet" "~"
-			(at 157.48 66.04 0)
-			(effects
-				(font
-					(size 1.27 1.27)
-				)
-				(hide yes)
-			)
-		)
-		(property "Description" ""
-			(at 157.48 66.04 0)
-			(effects
-				(font
-					(size 1.27 1.27)
-				)
-				(hide yes)
-			)
-		)
-		(pin "1"
-		)
-		(pin "2"
-		)
-		(instances
-			(project "guitarpreamp"
-				(path "/565fa02a-6c9c-4bdd-8ba2-36fe749429c4"
-					(reference "C12")
-					(unit 1)
-				)
-			)
-			(project "full_board_pico_seed"
-				(path "/e63e39d7-6ac0-4ffd-8aa3-1841a4541b55/6ec17984-49ce-45c2-b1f4-ed6e904b8c80"
-					(reference "C8")
+					(reference "R30")
 					(unit 1)
 				)
@@
 			(project "full_board_pico_seed"
 				(path "/e63e39d7-6ac0-4ffd-8aa3-1841a4541b55/6ec17984-49ce-45c2-b1f4-ed6e904b8c80"
-					(reference "C29")
-					(unit 1)
-				)
-			)
-		)
-	)
-	(symbol
-		(lib_id "Device:C_Polarized")
-		(at 157.48 58.42 270)
-		(unit 1)
-		(exclude_from_sim no)
-		(in_bom yes)
-		(on_board yes)
-		(dnp no)
-		(property "Reference" "C10"
-			(at 151.638 61.468 90)
-			(effects
-				(font
-					(size 1.27 1.27)
-				)
-			)
-		)
-		(property "Value" "10uF"
-			(at 152.4 59.69 90)
-			(effects
-				(font
-					(size 1.27 1.27)
-				)
-			)
-		)
-		(property "Footprint" "Capacitor_SMD:CP_Elec_4x4.5"
-			(at 153.67 59.3852 0)
-			(effects
-				(font
-					(size 1.27 1.27)
-				)
-				(hide yes)
-			)
-		)
-		(property "Datasheet" "~"
-			(at 157.48 58.42 0)
-			(effects
-				(font
-					(size 1.27 1.27)
-				)
-				(hide yes)
-			)
-		)
-		(property "Description" ""
-			(at 157.48 58.42 0)
-			(effects
-				(font
-					(size 1.27 1.27)
-				)
-				(hide yes)
-			)
-		)
-		(pin "1"
-		)
-		(pin "2"
-		)
-		(instances
-			(project "guitarpreamp"
-				(path "/565fa02a-6c9c-4bdd-8ba2-36fe749429c4"
-					(reference "C10")
-					(unit 1)
-				)
-			)
-			(project "full_board_pico_seed"
-				(path "/e63e39d7-6ac0-4ffd-8aa3-1841a4541b55/6ec17984-49ce-45c2-b1f4-ed6e904b8c80"
-					(reference "C24")
+					(reference "C23")
 					(unit 1)
 				)
@@
 			(project "full_board_pico_seed"
 				(path "/e63e39d7-6ac0-4ffd-8aa3-1841a4541b55/6ec17984-49ce-45c2-b1f4-ed6e904b8c80"
-					(reference "C30")
+					(reference "C24")
 					(unit 1)
 				)
@@
 			(project "full_board_pico_seed"
 				(path "/e63e39d7-6ac0-4ffd-8aa3-1841a4541b55/6ec17984-49ce-45c2-b1f4-ed6e904b8c80"
-					(reference "R32")
+					(reference "R28")
 					(unit 1)
 				)
@@
 		(on_board yes)
 		(dnp no)
-		(property "Reference" "C5"
+		(property "Reference" "C7"
 			(at 212.598 83.566 0)
 			(effects
@@
 			(project "full_board_pico_seed"
 				(path "/e63e39d7-6ac0-4ffd-8aa3-1841a4541b55/6ec17984-49ce-45c2-b1f4-ed6e904b8c80"
-					(reference "C5")
+					(reference "C7")
 					(unit 1)
 				)
@@
 		(on_board yes)
 		(dnp no)
-		(property "Reference" "TP4"
+		(property "Reference" "TP5"
 			(at 203.2 68.834 90)
 			(effects
@@
 			(project "full_board_pico_seed"
 				(path "/e63e39d7-6ac0-4ffd-8aa3-1841a4541b55/6ec17984-49ce-45c2-b1f4-ed6e904b8c80"
-					(reference "TP4")
-					(unit 1)
-				)
+					(reference "TP5")
+					(unit 1)
+				)
