File: schematics/full_board_pico_seed/full_board_pico_seed.kicad_pcb (KiCad board)
At the start: 4 copper layers, 128.3 x 74.9 mm, 144 parts, among them J1 XLR3, J10 Conn_02x03_Odd_Even, J2 Aux In, J3 Conn_01x02_Pin, J4 Conn_01x03_Female, J5 XLR3, J6 XLR3, J7 Conn_02x20_Odd_Even, J8 Conn_01x03, J9 Conn_01x02_Male, P1 25k, P2 25k, P3 25k, SW1 Stompbutton 1, SW2 Stompbutton 2, SW3 Stompbutton 3, SW4 Exit, SW5 Enter, U1 OPA134, U10 128X64 OLED Display, U2 OPA2342, U3 OPA4342, U4 LM4881M/NOPB, U5 PCM3060, U6 LM1117DT-5.0, U7 ATmega88A-A, U8 AP63205WU, U9 24LC128, X1 SG-5032CAN 12.288MHz

Commit message: schematic change
Parts:
- removed the C24 at (106.7, 88.9)
- removed the C6 at (100.3, 75.6)
- removed the C8 at (112.3, 74.4)
- removed the C9 at (105.7, 72.4)
- removed the R16 at (135.2, 68.7)
- removed the R23 at (145.3, 68.7)
- removed the R24 at (149.6, 68.7)
- removed the R8 at (135.2, 70.6)
- removed TP_ADC1, TP_ADC2, TP_PD1: ~, TestPoint:TestPoint_Pad_D1.5mm
- added TP_ADC6: ~, TestPoint:TestPoint_Pad_D1.5mm, F.Cu at (111.0, 119.4)
- added TP_ADC7: ~, TestPoint:TestPoint_Pad_D1.5mm, F.Cu at (111.0, 110.7)
- added TP_PD7: ~, TestPoint:TestPoint_Pad_D1.5mm, F.Cu at (98.8, 132.6)
- C11: renamed from C12; value 10uF -> 4.7uF; footprint Capacitor_SMD:CP_Elec_4x4.5 -> Capacitor_SMD:CP_Elec_5x5.4
- C12: renamed from C13; value 10uF -> 4.7uF; footprint Capacitor_SMD:CP_Elec_4x4.5 -> Capacitor_SMD:CP_Elec_5x5.4
- C14: renamed from C16; value 10uF -> 4.7uF; footprint Capacitor_SMD:CP_Elec_4x4.5 -> Capacitor_SMD:CP_Elec_5x5.4
- C15: renamed from C18; value 10uF -> 4.7uF; footprint Capacitor_SMD:CP_Elec_4x4.5 -> Capacitor_SMD:CP_Elec_5x5.4
- H1: renamed from H4; footprint MountingHole:MountingHole_3.2mm_M3 -> MountingHole:MountingHole_4.3mm_M4
- H2: renamed from H1; footprint MountingHole:MountingHole_3.2mm_M3 -> MountingHole:MountingHole_4.3mm_M4
- H3: renamed from H2; footprint MountingHole:MountingHole_3.2mm_M3 -> MountingHole:MountingHole_4.3mm_M4
- H4: renamed from H3; footprint MountingHole:MountingHole_3.2mm_M3 -> MountingHole:MountingHole_4.3mm_M4
- U1: value OPA134 -> OPA1602
- moved TP_PD5 15.2 mm to (99.3, 117.3)
- moved TP2 11.8 mm to (74.9, 85.7)
- moved TP_PD4 9.49 mm to (96.8, 108.2)
- moved R1 9.16 mm to (76.8, 80.6), turned to 90 degrees
- moved R2 7.01 mm to (82.8, 78.2), turned to 180 degrees
- moved R31 6.76 mm to (101.1, 91.8)
- moved J4 6.71 mm to (118.4, 66.2)
- moved H1 6.13 mm to (74.3, 70.1)
- moved C6 6.04 mm to (94.7, 74.9)
- moved C5 5.85 mm to (101.3, 86.9)
- moved R6 5.85 mm to (103.9, 86.9)
- moved TP1 5.57 mm to (87.9, 84.3)
- moved R3 4.96 mm to (74.9, 80.6)
- moved RV2 4.92 mm to (106.4, 66.2)
- moved R15 4.56 mm to (134.8, 69.6), turned to 0 degrees
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- renumbered C3 to C1, C15 to C10, C14 to C13, C17 to C16, C19 to C17, C21 to C18, C20 to C19, C23 to C20, C22 to C21, C27 to C22, C29 to C23, C30 to C24, C26 to C25, C28 to C26, C31 to C27, C32 to C28, C33 to C29, C1 to C3, C7 to C4, C25 to C5, C4 to C6, C5 to C7, C10 to C8, C11 to C9, D12 to D2, D11 to D3, D10 to D4, D8 to D5, D7 to D6, J3 to J2, J6 to J3, J2 to J4, J4 to J5, J5 to J6, R4 to R1, R7 to R10, R17 to R11, R11 to R12, R12 to R13, R9 to R14, R14 to R15, R15 to R16, R18 to R17, R20 to R18, R26 to R19, R5 to R2, R22 to R20, R28 to R21, R29 to R22, R21 to R23, R27 to R24, R30 to R26, R31 to R27, R32 to R28, R2 to R29, R33 to R30, R35 to R31, R36 to R32, R37 to R33, R39 to R34, R42 to R35, R43 to R36, R38 to R37, R41 to R38, R40 to R39, R1 to R4, R45 to R40, R46 to R41, R47 to R42, R44 to R43, R6 to R5, R34 to R6, R10 to R7, R19 to R8, R13 to R9, TP3 to TP1, TP7 to TP10, TP1 to TP3, TP5 to TP4, TP4 to TP5, TP8 to TP7, TP9 to TP8, TP10 to TP9
Connections:
- C3 pad 1: /Analog Preamp/VCom -> Net-(U1B--)
- C4 pad 2: Net-(C7-Pad2) -> /Analog Preamp/Mic
- C5 pad 2: Net-(C25-Pad2) -> Net-(C5-Pad2)
- R1 pad 2: Net-(R4-Pad2) -> Net-(R1-Pad2)
- R2 pad 2: Net-(R4-Pad2) -> Net-(R1-Pad2)
- R29 pad 1: /Analog Preamp/VCom -> Net-(U1B--)
- R5 pad 1: /Analog Preamp/VCom -> Net-(U1B--)
- R6 pad 2: Net-(C25-Pad2) -> Net-(C5-Pad2)
- RV1 pad 1: Net-(C7-Pad2) -> /Analog Preamp/Mic
- RV2 pad 1: Net-(C6-Pad2) -> Net-(C5-Pad2)
- RV2 pad 3: GND -> Net-(U1B--)
- TP1 pad 1: /Analog Preamp/VCom -> Net-(U1B--)
- TP2 pad 1: Net-(R4-Pad2) -> Net-(R1-Pad2)
- TP_PD3 pad 1: Net-(U7-PD4) -> Net-(U7-PD3)
- TP_PD4 pad 1: Net-(U7-PD5) -> Net-(U7-PD4)
- TP_PD5 pad 1: Net-(U7-PD7) -> Net-(U7-PD5)
- U1 pad 1: unconnected-(U1-BAL-Pad1) -> Net-(R1-Pad2)
- U1 pad 5: unconnected-(U1-COMP-Pad5) -> /Analog Preamp/VCom
- U1 pad 6: Net-(R4-Pad2) -> Net-(U1B--)
- U1 pad 7: 5V -> Net-(U1B--)
- U1 pad 8: unconnected-(U1-C/B-Pad8) -> 5V
- U2 pad 1: Net-(C7-Pad2) -> /Analog Preamp/Mic
- U2 pad 3: /Analog Preamp/VCom -> Net-(U1B--)
- U2 pad 7: Net-(C25-Pad2) -> Net-(C5-Pad2)
- U3 pad 10: /Analog Preamp/VCom -> Net-(U1B--)
- U3 pad 12: /Analog Preamp/VCom -> Net-(U1B--)
- U3 pad 3: /Analog Preamp/VCom -> Net-(U1B--)
- U3 pad 5: /Analog Preamp/VCom -> Net-(U1B--)
- U5 pad 25: Net-(U5-V_{IN}L) -> /Analog Preamp/HiZ
- U5 pad 26: Net-(U5-V_{IN}R) -> /Analog Preamp/Mic
Routing:
- net Net-(U1B--): track 0.00 -> 106.8 mm, vias 0 -> 4
- net /Analog Preamp/VCom: track 97.6 -> 43.8 mm, vias 6 -> 2
- net Net-(C7-Pad2): track 38.5 -> 0.00 mm
- net /Analog Preamp/Mic: track 13.3 -> 44.5 mm, vias 0 -> 2
- net Net-(C5-Pad2): track 0.00 -> 25.3 mm
- net Net-(U5-V_{IN}R): track 24.4 -> 0.00 mm, vias 2 -> 0
- net Net-(C25-Pad2): track 20.9 -> 0.00 mm
- net /Analog Preamp/HiZ: track 21.5 -> 37.4 mm
- net Net-(R1-Pad2): track 0.00 -> 14.3 mm
- net Net-(U2B-+): track 31.5 -> 19.4 mm, vias 0 -> 2
- net GND: track 158.5 -> 146.6 mm, vias 25 -> 23
- net Net-(U5-V_{IN}L): track 11.9 -> 0.00 mm
- net Net-(R4-Pad2): track 11.2 -> 0.00 mm
- net Net-(C6-Pad2): track 10.8 -> 0.00 mm
- net Net-(U1A--): track 12.9 -> 4.56 mm
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