File: schematics/full_board_pico_seed/full_board_pico_seed.kicad_sch (KiCad schematic)
At the start: 32 parts, among them J7 Conn_02x20_Odd_Even, J8 Conn_01x03, J9 Conn_01x02_Male, P1 25k, P2 25k, P3 25k, SW4 Exit, SW5 Enter, U10 128X64 OLED Display, U6 LM1117DT-5.0, U8 AP63205WU

Commit message: schematic change
Parts:
- H1: renamed from H4; footprint MountingHole:MountingHole_3.2mm_M3 -> MountingHole:MountingHole_4.3mm_M4
- H2: renamed from H1; footprint MountingHole:MountingHole_3.2mm_M3 -> MountingHole:MountingHole_4.3mm_M4
- H3: renamed from H2; footprint MountingHole:MountingHole_3.2mm_M3 -> MountingHole:MountingHole_4.3mm_M4
- H4: renamed from H3; footprint MountingHole:MountingHole_3.2mm_M3 -> MountingHole:MountingHole_4.3mm_M4
- renumbered C21 to C18, C23 to C20, C22 to C21, C26 to C25, C31 to C27, C32 to C28, C33 to C29, D8 to D5, D7 to D6, R30 to R26, R31 to R27, R36 to R32, R37 to R33, R45 to R40, R46 to R41, R47 to R42
Changed lines of the file:
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@@
 		(dnp no)
 		(fields_autoplaced yes)
-		(property "Reference" "H4"
+		(property "Reference" "H1"
 			(at 134.62 192.2053 0)
 			(effects
@@
 			)
 		)
-		(property "Footprint" "MountingHole:MountingHole_3.2mm_M3"
+		(property "Footprint" "MountingHole:MountingHole_4.3mm_M4"
 			(at 132.08 193.04 0)
 			(effects
@@
 			(project "full_board_pico_seed"
 				(path "/e63e39d7-6ac0-4ffd-8aa3-1841a4541b55"
-					(reference "H4")
+					(reference "H1")
 					(unit 1)
 				)
@@
 		(on_board yes)
 		(dnp no)
-		(property "Reference" "R30"
+		(property "Reference" "R26"
 			(at 63.5 109.22 0)
 			(effects
@@
 			(project "full_board_pico_seed"
 				(path "/e63e39d7-6ac0-4ffd-8aa3-1841a4541b55"
-					(reference "R30")
+					(reference "R26")
 					(unit 1)
 				)
@@
 		(dnp no)
 		(fields_autoplaced yes)
-		(property "Reference" "C31"
+		(property "Reference" "C27"
 			(at 55.88 147.32 0)
 			(effects
@@
 			(project "full_board_pico_seed"
 				(path "/e63e39d7-6ac0-4ffd-8aa3-1841a4541b55"
-					(reference "C31")
+					(reference "C27")
 					(unit 1)
 				)
@@
 		(on_board yes)
 		(dnp no)
-		(property "Reference" "D8"
+		(property "Reference" "D5"
 			(at 153.67 172.72 0)
 			(effects
@@
 			(project "full_board_pico_seed"
 				(path "/e63e39d7-6ac0-4ffd-8aa3-1841a4541b55"
-					(reference "D8")
+					(reference "D5")
 					(unit 1)
 				)
@@
 		(dnp no)
 		(fields_autoplaced yes)
-		(property "Reference" "R37"
+		(property "Reference" "R33"
 			(at 54.61 130.81 0)
 			(effects
@@
 			(project "full_board_pico_seed"
 				(path "/e63e39d7-6ac0-4ffd-8aa3-1841a4541b55"
-					(reference "R37")
+					(reference "R33")
 					(unit 1)
 				)
@@
 		(dnp no)
 		(fields_autoplaced yes)
-		(property "Reference" "R47"
+		(property "Reference" "R42"
 			(at 95.25 171.45 0)
 			(effects
@@
 			(project "full_board_pico_seed"
 				(path "/e63e39d7-6ac0-4ffd-8aa3-1841a4541b55"
-					(reference "R47")
+					(reference "R42")
 					(unit 1)
 				)
@@
 		(on_board yes)
 		(dnp no)
-		(property "Reference" "C21"
+		(property "Reference" "C18"
 			(at 63.5 115.57 0)
 			(effects
@@
 			(project "full_board_pico_seed"
 				(path "/e63e39d7-6ac0-4ffd-8aa3-1841a4541b55"
-					(reference "C21")
+					(reference "C18")
 					(unit 1)
 				)
@@
 		(dnp no)
 		(fields_autoplaced yes)
-		(property "Reference" "R36"
+		(property "Reference" "R32"
 			(at 54.61 139.7 0)
 			(effects
@@
 			(project "full_board_pico_seed"
 				(path "/e63e39d7-6ac0-4ffd-8aa3-1841a4541b55"
-					(reference "R36")
+					(reference "R32")
 					(unit 1)
 				)
@@
 		(on_board yes)
 		(dnp no)
-		(property "Reference" "C22"
+		(property "Reference" "C21"
 			(at 240.411 74.4763 0)
 			(effects
@@
 			(project "full_board_pico_seed"
 				(path "/e63e39d7-6ac0-4ffd-8aa3-1841a4541b55"
-					(reference "C22")
+					(reference "C21")
 					(unit 1)
 				)
@@
 		(dnp no)
 		(fields_autoplaced yes)
-		(property "Reference" "H3"
+		(property "Reference" "H4"
 			(at 160.02 183.3153 0)
 			(effects
@@
 			)
 		)
-		(property "Footprint" "MountingHole:MountingHole_3.2mm_M3"
+		(property "Footprint" "MountingHole:MountingHole_4.3mm_M4"
 			(at 157.48 184.15 0)
 			(effects
@@
 			(project "full_board_pico_seed"
 				(path "/e63e39d7-6ac0-4ffd-8aa3-1841a4541b55"
-					(reference "H3")
+					(reference "H4")
 					(unit 1)
 				)
@@
 		(on_board yes)
 		(dnp no)
-		(property "Reference" "C32"
+		(property "Reference" "C28"
 			(at 265.811 89.7163 0)
 			(effects
@@
 			(project "full_board_pico_seed"
 				(path "/e63e39d7-6ac0-4ffd-8aa3-1841a4541b55"
-					(reference "C32")
+					(reference "C28")
 					(unit 1)
 				)
@@
 		(on_board yes)
 		(dnp no)
-		(property "Reference" "R31"
+		(property "Reference" "R27"
 			(at 60.96 101.6 0)
 			(effects
@@
 			(project "full_board_pico_seed"
 				(path "/e63e39d7-6ac0-4ffd-8aa3-1841a4541b55"
-					(reference "R31")
+					(reference "R27")
 					(unit 1)
 				)
@@
 		(on_board yes)
 		(dnp no)
-		(property "Reference" "C33"
+		(property "Reference" "C29"
 			(at 251.46 100.33 0)
 			(effects
@@
 			(project "full_board_pico_seed"
 				(path "/e63e39d7-6ac0-4ffd-8aa3-1841a4541b55"
-					(reference "C33")
+					(reference "C29")
 					(unit 1)
 				)
@@
 		(on_board yes)
 		(dnp no)
-		(property "Reference" "R46"
+		(property "Reference" "R41"
 			(at 165.1 167.64 90)
 			(effects
@@
 			(project "full_board_pico_seed"
 				(path "/e63e39d7-6ac0-4ffd-8aa3-1841a4541b55"
-					(reference "R46")
+					(reference "R41")
 					(unit 1)
 				)
@@
 		(on_board yes)
 		(dnp no)
-		(property "Reference" "R45"
+		(property "Reference" "R40"
 			(at 166.37 162.56 90)
 			(effects
@@
 			(project "full_board_pico_seed"
 				(path "/e63e39d7-6ac0-4ffd-8aa3-1841a4541b55"
-					(reference "R45")
+					(reference "R40")
 					(unit 1)
 				)
@@
 		(dnp no)
 		(fields_autoplaced yes)
-		(property "Reference" "C26"
+		(property "Reference" "C25"
 			(at 264.16 74.0409 0)
 			(effects
@@
 			(project "full_board_pico_seed"
 				(path "/e63e39d7-6ac0-4ffd-8aa3-1841a4541b55"
-					(reference "C26")
+					(reference "C25")
 					(unit 1)
 				)
@@
 		(on_board yes)
 		(dnp no)
-		(property "Reference" "C23"
+		(property "Reference" "C20"
 			(at 218.821 98.6063 0)
 			(effects
@@
 			(project "full_board_pico_seed"
 				(path "/e63e39d7-6ac0-4ffd-8aa3-1841a4541b55"
-					(reference "C23")
+					(reference "C20")
 					(unit 1)
 				)
@@
 		(dnp no)
 		(fields_autoplaced yes)
-		(property "Reference" "H2"
+		(property "Reference" "H3"
 			(at 160.02 174.4253 0)
 			(effects
@@
 			)
 		)
-		(property "Footprint" "MountingHole:MountingHole_3.2mm_M3"
+		(property "Footprint" "MountingHole:MountingHole_4.3mm_M4"
 			(at 157.48 175.26 0)
 			(effects
@@
 			(project "full_board_pico_seed"
 				(path "/e63e39d7-6ac0-4ffd-8aa3-1841a4541b55"
-					(reference "H2")
+					(reference "H3")
 					(unit 1)
 				)
@@
 		(on_board yes)
 		(dnp no)
-		(property "Reference" "D7"
+		(property "Reference" "D6"
 			(at 152.4 162.56 0)
 			(effects
@@
 			(project "full_board_pico_seed"
 				(path "/e63e39d7-6ac0-4ffd-8aa3-1841a4541b55"
-					(reference "D7")
+					(reference "D6")
 					(unit 1)
 				)
@@
 		(dnp no)
 		(fields_autoplaced yes)
-		(property "Reference" "H1"
+		(property "Reference" "H2"
 			(at 160.02 192.2053 0)
 			(effects
@@
 			)
 		)
-		(property "Footprint" "MountingHole:MountingHole_3.2mm_M3"
+		(property "Footprint" "MountingHole:MountingHole_4.3mm_M4"
 			(at 157.48 193.04 0)
 			(effects
@@
 			(project "full_board_pico_seed"
 				(path "/e63e39d7-6ac0-4ffd-8aa3-1841a4541b55"
-					(reference "H1")
+					(reference "H2")
 					(unit 1)
 				)

Commit message: updated schematic
Connections:
- net 3V3: now also U10.2 (3.3V); no longer U10.6 (3.3V)
- net GND: now also J8.1 (Pin_1), U10.1 (Ground); no longer J8.2 (Pin_2), U10.7 (Ground)
- net at R32.1, R33.2: now also J8.2 (Pin_2); no longer J8.1 (Pin_1)
- net at J7.12 (Pin_12), R42.1: now also U10.3 (Reset); no longer U10.5 (Reset)
- net UI Controller/prog_miso: now reaches J7.15 (Pin_15)
- net UI Controller/prog_reset: now reaches J7.17 (Pin_17)
- net at J7.4 (Pin_4): now also U10.7 (DC); no longer U10.1 (DC)
- net UI Controller/prog_mosi: now reaches J7.6 (Pin_6)
- net UI Controller/prog_mosi: now also U10.6 (Data); no longer U10.2 (Data)
- net UI Controller/prog_sck: now reaches J7.8 (Pin_8)
- net UI Controller/prog_sck: now also U10.5 (SCLK); no longer U10.3 (SCLK)
- no-connect marks 14 -> 12
Other:
- sheet UI Controller ports: added prog_miso, prog_mosi, prog_reset, prog_sck; removed none
- moved on the sheet: R42
