File: schematics/adapter_pico/adapter_pico.kicad_sch (KiCad schematic)
At the start: 2 parts, among them J1 Conn_02x20_Odd_Even, U2 Pico

Commit message: daisy seed adapter board: initial layout
Connections:
- net GND: now also J1.20 (Pin_20); no longer J1.39 (Pin_39)
Changed lines of the file:
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@@
   (no_connect (at 114.3 102.87))
   (no_connect (at 114.3 87.63))
+  (no_connect (at 114.3 110.49))
   (no_connect (at 114.3 90.17))
   (no_connect (at 135.89 137.16))
@@
   (no_connect (at 135.89 132.08))
   (no_connect (at 135.89 149.86))
-  (no_connect (at 127 85.09))
   (no_connect (at 100.33 127))
   (no_connect (at 127 107.95))
@@
     )
   )
-  (symbol (lib_id "power:GND") (at 114.3 110.49 270) (unit 1)
-    (in_bom yes) (on_board yes) (dnp no) (fields_autoplaced)
-    (property "Reference" "#PWR02" (at 107.95 110.49 0)
-      (effects (font (size 1.27 1.27)) hide)
-    )
-    (property "Value" "GND" (at 110.49 110.49 90)
+  (symbol (lib_id "power:GND") (at 127 85.09 90) (unit 1)
+    (in_bom yes) (on_board yes) (dnp no) (fields_autoplaced)
+    (property "Reference" "#PWR02" (at 133.35 85.09 0)
+      (effects (font (size 1.27 1.27)) hide)
+    )
+    (property "Value" "GND" (at 130.81 85.09 90)
       (effects (font (size 1.27 1.27)) (justify right))
     )
-    (property "Footprint" "" (at 114.3 110.49 0)
-      (effects (font (size 1.27 1.27)) hide)
-    )
-    (property "Datasheet" "" (at 114.3 110.49 0)
-      (effects (font (size 1.27 1.27)) hide)
-    )
+    (property "Footprint" "" (at 127 85.09 0)
+      (effects (font (size 1.27 1.27)) hide)
+    )
+    (property "Datasheet" "" (at 127 85.09 0)
+      (effects (font (size 1.27 1.27)) hide)
+    )

Commit message: correct codec sdin and sdout directions
Connections:
- net at J1.13 (Pin_13): now also U2.16 (GPIO12); no longer U2.12 (GPIO9)
- net at J1.5 (Pin_5): now also U2.12 (GPIO9); no longer U2.16 (GPIO12)
Changed lines of the file:
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@@
+    (stroke (width 0) (type default))
+  )
+  (wire (pts (xy 81.28 152.4) (xy 100.33 152.4))
     (stroke (width 0) (type default))
   )
   (wire (pts (xy 73.66 74.93) (xy 73.66 157.48))
-    (stroke (width 0) (type default))
-  )
-  (wire (pts (xy 86.36 77.47) (xy 86.36 152.4))
     (stroke (width 0) (type default))
   )
@@
   )
   (wire (pts (xy 162.56 97.79) (xy 162.56 147.32))
-    (stroke (width 0) (type default))
-  )
-  (wire (pts (xy 81.28 162.56) (xy 100.33 162.56))
     (stroke (width 0) (type default))
   )
@@
   )
   (wire (pts (xy 93.98 69.85) (xy 93.98 137.16))
+    (stroke (width 0) (type default))
+  )
+  (wire (pts (xy 86.36 77.47) (xy 86.36 162.56))
     (stroke (width 0) (type default))
   )
@@
   )
   (wire (pts (xy 160.02 87.63) (xy 160.02 152.4))
-    (stroke (width 0) (type default))
-  )
-  (wire (pts (xy 86.36 152.4) (xy 100.33 152.4))
     (stroke (width 0) (type default))
   )
@@
     (stroke (width 0) (type default))
   )
-  (wire (pts (xy 81.28 67.31) (xy 81.28 162.56))
+  (wire (pts (xy 81.28 67.31) (xy 81.28 152.4))
     (stroke (width 0) (type default))
   )
@@
     (stroke (width 0) (type default))
   )
+  (wire (pts (xy 86.36 162.56) (xy 100.33 162.56))
+    (stroke (width 0) (type default))
+  )

Commit message: avr flasher: schematic changes
Connections:
- net at J1.15 (Pin_15): now also U2.26 (GPIO20)
- net at J1.17 (Pin_17): now also U2.17 (GPIO13)
- net at J1.18 (Pin_18): now also U2.4 (GPIO2); no longer U2.26 (GPIO20)
- no-connect marks 27 -> 23
